File: 02 Electrical/BicycleRimPowerSupply - Simulation/BicycleRimPowerSupply.kicad_sch (KiCad schematic)
At the start: 14 parts

Commit message: Simulations added
Parts:
- gave numbers to parts that had none: 4
- renumbered D2 to D5, D3 to D6, D4 to D7
Changed lines of the file:
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@@
   (symbol (lib_id "Diode:1N4002") (at 116.84 52.07 0) (unit 1)
     (in_bom yes) (on_board yes) (fields_autoplaced)
-    (property "Reference" "D2" (id 0) (at 116.84 45.085 0))
+    (property "Reference" "D5" (id 0) (at 116.84 45.085 0))
     (property "Value" "1N4002" (id 1) (at 116.84 47.625 0))
     (property "Footprint" "Diode_THT:D_T-1_P5.08mm_Horizontal" (id 2) (at 116.84 56.515 0)
@@
   (symbol (lib_id "pspice:DIODE") (at 84.455 69.85 90) (unit 1)
     (in_bom yes) (on_board yes) (fields_autoplaced)
-    (property "Reference" "D?" (id 0) (at 88.265 68.5799 90)
+    (property "Reference" "D3" (id 0) (at 88.265 68.5799 90)
       (effects (font (size 1.27 1.27)) (justify right))
     )
@@
   (symbol (lib_id "pspice:DIODE") (at 73.66 69.85 90) (unit 1)
     (in_bom yes) (on_board yes) (fields_autoplaced)
-    (property "Reference" "D?" (id 0) (at 77.47 68.5799 90)
+    (property "Reference" "D1" (id 0) (at 77.47 68.5799 90)
       (effects (font (size 1.27 1.27)) (justify right))
     )
@@
   (symbol (lib_id "Device:LED") (at 163.83 69.215 90) (unit 1)
     (in_bom yes) (on_board yes) (fields_autoplaced)
-    (property "Reference" "D4" (id 0) (at 167.64 69.5324 90)
+    (property "Reference" "D7" (id 0) (at 167.64 69.5324 90)
       (effects (font (size 1.27 1.27)) (justify right))
     )
@@
   (symbol (lib_id "pspice:DIODE") (at 73.66 81.915 90) (unit 1)
     (in_bom yes) (on_board yes) (fields_autoplaced)
-    (property "Reference" "D?" (id 0) (at 77.47 80.6449 90)
+    (property "Reference" "D2" (id 0) (at 77.47 80.6449 90)
       (effects (font (size 1.27 1.27)) (justify right))
     )
@@
   (symbol (lib_id "pspice:DIODE") (at 84.455 81.915 90) (unit 1)
     (in_bom yes) (on_board yes) (fields_autoplaced)
-    (property "Reference" "D?" (id 0) (at 88.265 80.6449 90)
+    (property "Reference" "D4" (id 0) (at 88.265 80.6449 90)
       (effects (font (size 1.27 1.27)) (justify right))
     )
@@
   (symbol (lib_id "Diode:1N4002") (at 138.43 70.485 270) (unit 1)
     (in_bom yes) (on_board yes) (fields_autoplaced)
-    (property "Reference" "D3" (id 0) (at 141.605 69.2149 90)
+    (property "Reference" "D6" (id 0) (at 141.605 69.2149 90)
       (effects (font (size 1.27 1.27)) (justify left))
     )
@@
       (reference "C3") (unit 1) (value "1uF") (footprint "Capacitor_THT:C_Axial_L3.8mm_D2.6mm_P7.50mm_Horizontal")
     )
+    (path "/35a5af30-ea08-424c-b901-e20b3af59c99"
+      (reference "D1") (unit 1) (value "DIODE") (footprint "")
+    )
+    (path "/5ddfb6a2-cd16-4b75-922d-72269a46826b"
+      (reference "D2") (unit 1) (value "DIODE") (footprint "")
+    )
+    (path "/34392292-7065-417e-b176-902ff9b9f131"
+      (reference "D3") (unit 1) (value "DIODE") (footprint "")
+    )
+    (path "/5dfab41b-35e0-4bcc-964d-616bf1ed5c2b"
+      (reference "D4") (unit 1) (value "DIODE") (footprint "")
+    )
     (path "/217014c2-1ef3-4b3f-b89a-760756a34189"
-      (reference "D2") (unit 1) (value "1N4002") (footprint "Diode_THT:D_T-1_P5.08mm_Horizontal")
+      (reference "D5") (unit 1) (value "1N4002") (footprint "Diode_THT:D_T-1_P5.08mm_Horizontal")
     )
     (path "/af0141e3-a63e-4f45-a945-21b8388e2d2f"
-      (reference "D3") (unit 1) (value "1N4002") (footprint "Diode_THT:D_DO-41_SOD81_P10.16mm_Horizontal")
+      (reference "D6") (unit 1) (value "1N4002") (footprint "Diode_THT:D_DO-41_SOD81_P10.16mm_Horizontal")
     )
     (path "/5ca767fe-178d-4bd1-9a62-3311f61d1ae1"
-      (reference "D4") (unit 1) (value "LED") (footprint "")
-    )
-    (path "/34392292-7065-417e-b176-902ff9b9f131"
-      (reference "D?") (unit 1) (value "DIODE") (footprint "")
-    )
-    (path "/35a5af30-ea08-424c-b901-e20b3af59c99"
-      (reference "D?") (unit 1) (value "DIODE") (footprint "")
-    )
-    (path "/5ddfb6a2-cd16-4b75-922d-72269a46826b"
-      (reference "D?") (unit 1) (value "DIODE") (footprint "")
-    )
-    (path "/5dfab41b-35e0-4bcc-964d-616bf1ed5c2b"
-      (reference "D?") (unit 1) (value "DIODE") (footprint "")
+      (reference "D7") (unit 1) (value "LED") (footprint "")
     )
     (path "/3bc802c5-99dd-439b-849d-88d55fdb1923"
