File: 02 Electrical/Power supply with regulator/Power supply with regulator.kicad_sch (KiCad schematic)
At the start: 8 parts, among them U1 L7805

Commit message: Simulation added
Parts:
- C1: value 2000uF -> 1uF
- R1: footprint (none) -> TestPoint:TestPoint_2Pads_Pitch5.08mm_Drill1.3mm
- U1: footprint (none) -> Package_TO_SOT_SMD:SOT-223
- V1: value VSOURCE -> IN; footprint (none) -> TestPoint:TestPoint_2Pads_Pitch5.08mm_Drill1.3mm; Spice_Model dc 0 ac 40 sin(0 10 5) -> dc 0 ac 40 sin(0 40 15)
Other:
- title: (none) -> Bicycle rim power supply
- moved on the sheet: C1, D1, D2, D3, D4, R1, U1, V1
